Commit message: feat(examples): align cart-pole URDF with OpenAI Gym CartPole-v1 parameters
- Pole half-length: 0.2m → 0.5m (total 1.0m), matching Gym standard
- Pole inertia: mL²/12 = 0.00833 for uniform rod about COM
- Cart force: 20N → 10N (Gym standard)
- Cart limits: ±1.0m → ±2.4m (Gym termination threshold)
- Pole joint: revolute → continuous (no angle limits, termination in software)
- Remove all damping and friction (Gym has none)
- Gravity: 9.8 m/s² in tests (Gym standard)
- Update pendulum_viz visuals for longer pole and wider rail

Implements: 20260224-110336-dl-pipeline-test/02

Co-Authored-By: Claude Opus 4.6 <noreply@anthropic.com>

File: examples/urdf/cartpole.urdf (robot description, URDF)
Before this commit: robot cartpole, 3 links, 2 joints
Links:
- link pole: geometry collision cylinder length=1.0 radius=0.01; visual cylinder length=1.0 radius=0.01
- link rail: geometry visual box size=5.0 0.05 0.02
Joints:
- joint cart_slide: limit lower=-1.0 upper=1.0 effort=20 velocity=5 -> lower=-2.4 upper=2.4 effort=10 velocity=10
- joint pole_hinge: limit lower=-0.418 upper=0.418 effort=0 velocity=10 -> effort=0 velocity=20; type revolute -> continuous
