Commit message: feat(examples): upgrade quadruped to 3-DOF legs with full MPC locomotion
Upgrade URDF from 2-DOF (8 joints) to 3-DOF legs (12 joints) with hip
abduction. Rewrite headless and viz examples with complete MPC pipeline:
warmup knee-bending, stance J^T feedforward with per-joint gains,
Cartesian PD swing control, and Raibert foot placement.

Viz example adds egui control panel with gait selection, velocity/height
sliders (clamped to +/-0.5 m/s), and pipeline diagnostics. Both examples
use friction=1.0 for 2.5x margin over MPC mu=0.4, and swing max_force=30Nm
for 10cm step height clearance.

Co-Authored-By: Claude Opus 4.6 <noreply@anthropic.com>

File: examples/urdf/quadruped.urdf (robot description, URDF)
Before this commit: robot quadruped, 13 links, 12 joints
Links:
- added link fl_hip_link, mass 0.1; collision box size=0.04 0.04 0.04; visual box size=0.04 0.04 0.04
- added link fr_hip_link, mass 0.1; collision box size=0.04 0.04 0.04; visual box size=0.04 0.04 0.04
- added link rl_hip_link, mass 0.1; collision box size=0.04 0.04 0.04; visual box size=0.04 0.04 0.04
- added link rr_hip_link, mass 0.1; collision box size=0.04 0.04 0.04; visual box size=0.04 0.04 0.04
Joints:
- added joint fl_hip_ab: type revolute, parent body, child fl_hip_link, origin xyz=0.15 0.08 -0.05, axis 1 0 0, limit lower=-0.5 upper=0.5 effort=20 velocity=10
- added joint fr_hip_ab: type revolute, parent body, child fr_hip_link, origin xyz=0.15 -0.08 -0.05, axis 1 0 0, limit lower=-0.5 upper=0.5 effort=20 velocity=10
- added joint rl_hip_ab: type revolute, parent body, child rl_hip_link, origin xyz=-0.15 0.08 -0.05, axis 1 0 0, limit lower=-0.5 upper=0.5 effort=20 velocity=10
- added joint rr_hip_ab: type revolute, parent body, child rr_hip_link, origin xyz=-0.15 -0.08 -0.05, axis 1 0 0, limit lower=-0.5 upper=0.5 effort=20 velocity=10
- joint fl_hip_pitch: limit lower=-1.0 upper=1.0 effort=20 velocity=10 -> lower=-1.0 upper=1.0 effort=30 velocity=10; origin xyz=0.15 0.08 -0.05 -> xyz=0 0 0; parent body -> fl_hip_link
- joint fl_knee_pitch: limit lower=-2.5 upper=0.0 effort=20 velocity=10 -> lower=-2.5 upper=0.0 effort=30 velocity=10
- joint fr_hip_pitch: limit lower=-1.0 upper=1.0 effort=20 velocity=10 -> lower=-1.0 upper=1.0 effort=30 velocity=10; origin xyz=0.15 -0.08 -0.05 -> xyz=0 0 0; parent body -> fr_hip_link
- joint fr_knee_pitch: limit lower=-2.5 upper=0.0 effort=20 velocity=10 -> lower=-2.5 upper=0.0 effort=30 velocity=10
- joint rl_hip_pitch: limit lower=-1.0 upper=1.0 effort=20 velocity=10 -> lower=-1.0 upper=1.0 effort=30 velocity=10; origin xyz=-0.15 0.08 -0.05 -> xyz=0 0 0; parent body -> rl_hip_link
- joint rl_knee_pitch: limit lower=-2.5 upper=0.0 effort=20 velocity=10 -> lower=-2.5 upper=0.0 effort=30 velocity=10
- joint rr_hip_pitch: limit lower=-1.0 upper=1.0 effort=20 velocity=10 -> lower=-1.0 upper=1.0 effort=30 velocity=10; origin xyz=-0.15 -0.08 -0.05 -> xyz=0 0 0; parent body -> rr_hip_link
- joint rr_knee_pitch: limit lower=-2.5 upper=0.0 effort=20 velocity=10 -> lower=-2.5 upper=0.0 effort=30 velocity=10
