Commit message: feat(examples): add collision geometry and 2-finger gripper to six_dof_arm URDF
Implements: 20260228-201500-sensor-recording-arm/11

Co-Authored-By: Claude Opus 4.6 <noreply@anthropic.com>

File: examples/urdf/six_dof_arm.urdf (robot description, URDF)
Before this commit: robot six_dof_arm, 7 links, 6 joints
Links:
- added link finger_left, mass 0.02; collision box size=0.01 0.01 0.04; visual box size=0.01 0.01 0.04
- added link finger_right, mass 0.02; collision box size=0.01 0.01 0.04; visual box size=0.01 0.01 0.04
- added link gripper_base, mass 0.1; collision box size=0.06 0.04 0.02; visual box size=0.06 0.04 0.02
- link base: geometry collision cylinder length=0.1 radius=0.08; visual cylinder length=0.1 radius=0.08
- link elbow_link: geometry collision cylinder length=0.1 radius=0.03; visual cylinder length=0.1 radius=0.03
- link end_effector: geometry collision sphere radius=0.025; visual sphere radius=0.025
- link forearm: geometry collision cylinder length=0.2 radius=0.025; visual cylinder length=0.2 radius=0.025
- link shoulder_link: geometry collision cylinder length=0.2 radius=0.04; visual cylinder length=0.2 radius=0.04
- link upper_arm: geometry collision cylinder length=0.3 radius=0.035; visual cylinder length=0.3 radius=0.035
- link wrist_link: geometry collision cylinder length=0.06 radius=0.02; visual cylinder length=0.06 radius=0.02
Joints:
- added joint j_finger_left: type prismatic, parent gripper_base, child finger_left, origin xyz=0 0.015 0.01, axis 0 1 0, limit lower=0.0 upper=0.03 effort=10 velocity=0.1
- added joint j_finger_right: type prismatic, parent gripper_base, child finger_right, origin xyz=0 -0.015 0.01, axis 0 -1 0, limit lower=0.0 upper=0.03 effort=10 velocity=0.1
- added joint j_gripper_attach: type fixed, parent end_effector, child gripper_base, origin xyz=0 0 0.025
